Commit message: fwd added

File: catvehicle/urdf/catvehicle.urdf.xacro (robot description, xacro)
@@ -580,5 +580,5 @@
             <state_interface name="effort"/> -->
         </joint>
-        <joint name = 'back_left_wheel_joint'>
+        <joint name = 'front_left_wheel_joint'>
             <command_interface name = "velocity">
             <param name="min">-1000</param>
@@ -589,5 +589,5 @@
             <state_interface name="effort"/>
         </joint>
-        <joint name = 'back_right_wheel_joint'>
+        <joint name = 'front_right_wheel_joint'>
             <command_interface name = "velocity">
             <param name="min">-1000</param>
